File: elec/layout/default/bq24045dsqr.kicad_pcb (KiCad board)
At the start: 2 copper layers, 225.7 x 100.8 mm, 0 parts

Commit message: initial layout
Parts:
- added C1: Multilayer Ceramic Capacitors MLCC - SMD/SMT 1uF 6.3V 0402 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, lib:C0402, F.Cu at (164.5, 90.1)
- added C2: Multilayer Ceramic Capacitors MLCC - SMD/SMT 1uF 6.3V 0402 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, lib:C0402, F.Cu at (161.0, 90.1)
- added LED1: , lib:LED0603-RD, F.Cu at (159.7, 92.4)
- added LED2: , lib:LED0603-RD, F.Cu at (159.7, 89.5)
- added R1: Chip Resistor - Surface Mount 560Ohms ±5% 1/16W 0402 RoHS, lib:R0402, F.Cu at (161.0, 92.0)
- added R2: Chip Resistor - Surface Mount 120Ohms ±5% 1/16W 0402 RoHS, lib:R0402, F.Cu at (161.5, 93.5)
- added R3: Chip Resistor - Surface Mount 82Ohms ±5% 1/16W 0402 RoHS, lib:R0402, F.Cu at (161.6, 88.6)
- added U1: , lib:WSON-10_L2.0-W2.0-P0.40-BL-EP, F.Cu at (162.8, 90.8)
Routing:
- net vcc: track 0.00 -> 6.03 mm, vias 0 -> 2
- net gnd: track 0.00 -> 4.50 mm
- net vcc-1: track 0.00 -> 4.16 mm
- net gnd-1: track 0.00 -> 2.53 mm
- net iset: track 0.00 -> 1.99 mm
- net gnd-2: track 0.00 -> 1.55 mm
- net cathode: track 0.00 -> 1.46 mm
- net cathode-1: track 0.00 -> 1.38 mm

Commit message: update layout
Parts:
- removed LED1, LED2: , lib:LED0603-RD
- removed R2: Chip Resistor - Surface Mount 120Ohms ±5% 1/16W 0402 RoHS, lib:R0402
- removed R3: Chip Resistor - Surface Mount 82Ohms ±5% 1/16W 0402 RoHS, lib:R0402
- C1, C2: value Multilayer Ceramic Capacitors MLCC - SMD/SMT 1uF 6.3V 0402 RoHS -> 25V 1uF X5R ±10% 0402 Multilayer Ceramic Capacitors MLCC - SMD/SMT ROHS
- R1: value Chip Resistor - Surface Mount 560Ohms ±5% 1/16W 0402 RoHS -> 100mW Thick Film Resistors ±100ppm/℃ ±1% 604Ω 0402 Chip Resistor - Surface Mount ROHS
Connections:
- net gnd renamed ic-gnd
- net vcc renamed ic-vcc
- net vcc-1 renamed ic-vcc-1
- U1 pad 5: gnd-1 -> pg
- U1 pad 8: gnd-2 -> chg
Routing:
- net ic-vcc-1: track 4.16 -> 1.16 mm
- net gnd-1: track 2.53 -> 0.00 mm
- net gnd-2: track 1.55 -> 0.00 mm
- net cathode: track 1.46 -> 0.00 mm
- net cathode-1: track 1.38 -> 0.00 mm
- net iset: track 1.99 -> 2.76 mm

Commit message: Remove crud from layout
Other:
- board outline removed
- board text removed: "{{GITHASH}}"
